Commit message: added sliders to the base of the right arm to be able to move it around on the x-y plane via code

File: kinova_description/urdf/two_arm_m1n6s200_standalone.xacro (robot description, xacro)
@@ -38,7 +38,20 @@
     <origin xyz="-0.2 0 0" rpy="0 0 1.5707" />
   </joint>
-  <joint name="right_arm_attach" type="fixed">
-    <child link="right_arm_mount" />
-    <parent link="root" />
+<!--  <joint name="right_arm_attach" type="fixed">-->
+<!--    <child link="right_arm_mount" />-->
+<!--    <parent link="root" />-->
+<!--    <origin xyz="0.2 0 0" rpy="0 0 1.5707" />-->
+<!--  </joint>-->
+  <joint name="right_arm_slider_x" type="prismatic">
+    <parent link="root"/>
+    <child link="right_arm_mount_inner"/>
+    <limit effort="1000.0" lower="-0.38" upper="0" velocity="0.5"/>
+    <origin xyz="0.2 0 0" rpy="0 0 0" />
+  </joint>
+  <link name="right_arm_mount_inner"/>
+  <joint name="right_arm_slider_y" type="prismatic">
+    <parent link="right_arm_mount_inner"/>
+    <child link="right_arm_mount"/>
+    <limit effort="1000.0" lower="-0.38" upper="0" velocity="0.5"/>
     <origin xyz="0.2 0 0" rpy="0 0 1.5707" />
   </joint>

Commit message: add more robot statused

File: kinova_description/urdf/two_arm_m1n6s200_standalone.xacro (robot description, xacro)
@@ -36,12 +36,13 @@
     <child link="left_arm_mount" />
     <parent link="root" />
-    <origin xyz="-0.2 0 0" rpy="0 0 1.5707" />
+    <origin xyz="-0.4 0 0" rpy="0 0 1.5707" />
   </joint>
-<!--  <joint name="right_arm_attach" type="fixed">-->
-<!--    <child link="right_arm_mount" />-->
-<!--    <parent link="root" />-->
-<!--    <origin xyz="0.2 0 0" rpy="0 0 1.5707" />-->
-<!--  </joint>-->
-  <joint name="right_arm_slider_x" type="prismatic">
+ <joint name="right_arm_attach" type="fixed">
+   <child link="right_arm_mount" />
+   <parent link="root" />
+   <origin xyz="0.4 0 0" rpy="0 0 1.5707" />
+ </joint>
+  <!-- to create a prismatic joint to move the right arm around -->
+  <!-- <joint name="right_arm_slider_x" type="prismatic">
     <parent link="root"/>
     <child link="right_arm_mount_inner"/>
@@ -55,5 +56,5 @@
     <limit effort="1000.0" lower="-0.38" upper="0" velocity="0.5"/>
     <origin xyz="0.2 0 0" rpy="0 0 1.5707" />
-  </joint>
+  </joint> -->
   <xacro:m1n6s200  base_parent="left_arm_mount" prefix="left"/>
   <xacro:m1n6s200  base_parent="right_arm_mount" prefix="right"/>
